Commit message: add station

File: src/wms_description/urdf/wms_robot.urdf.xacro (robot description, xacro)
@@ -1,335 +1,323 @@
 <?xml version="1.0"?>
 <robot xmlns:xacro="http://www.ros.org/wiki/xacro" name="wms_robot">
-<!-- ====================================================== -->
-<!-- GAZEBO LIDAR SENSOR                                    -->
-<!-- ====================================================== -->
-<gazebo reference="lidar_link">
+  <!-- ====================================================== -->
+  <!-- ROBOT PARAMETERS                                       -->
+  <!-- ====================================================== -->
+  <xacro:property name="base_length" value="0.80"/>
+  <xacro:property name="base_width" value="0.60"/>
+  <xacro:property name="base_height" value="0.20"/>
+  <xacro:property name="base_mass" value="50.0"/>
+  <xacro:property name="wheel_radius" value="0.10"/>
+  <xacro:property name="wheel_width" value="0.05"/>
+  <xacro:property name="wheel_separation" value="0.65"/>
+  <xacro:property name="wheel_mass" value="2.0"/>
+  <xacro:property name="caster_radius" value="0.05"/>
+  <xacro:property name="caster_mass" value="0.5"/>
+  <xacro:property name="lidar_radius" value="0.05"/>
+  <xacro:property name="lidar_height" value="0.04"/>
+  <xacro:property name="lidar_mass" value="0.2"/>
+  <xacro:property name="imu_mass" value="0.05"/>
+  <!-- ====================================================== -->
+  <!-- BASE FOOTPRINT                                         -->
+  <!-- ====================================================== -->
+  <link name="base_footprint"/>
+  <!-- ====================================================== -->
+  <!-- BASE LINK                                              -->
+  <!-- ====================================================== -->
+  <link name="base_link">
+    <visual>
+      <geometry>
+        <box size="${base_length} ${base_width} ${base_height}"/>
+      </geometry>
+      <material name="blue">
+        <color rgba="0.1 0.3 0.8 1"/>
+      </material>
+    </visual>
+    <collision>
+      <geometry>
+        <box size="${base_length} ${base_width} ${base_height}"/>
+      </geometry>
+    </collision>
+    <inertial>
+      <mass value="${base_mass}"/>
+      <inertia
+        ixx="1.67"
+        ixy="0.0"
+        ixz="0.0"
+        iyy="2.83"
+        iyz="0.0"
+        izz="4.17"/>
+    </inertial>
+  </link>
+  <joint name="base_footprint_joint" type="fixed">
+    <parent link="base_footprint"/>
+    <child link="base_link"/>
+    <origin xyz="0 0 0.20" rpy="0 0 0"/>
+  </joint>
+  <!-- ====================================================== -->
+  <!-- LEFT DRIVE WHEEL                                       -->
+  <!-- ====================================================== -->
+  <link name="left_wheel_link">
+    <visual>
+      <geometry>
+        <cylinder radius="${wheel_radius}" length="${wheel_width}"/>
+      </geometry>
+      <material name="black">
+        <color rgba="0.05 0.05 0.05 1"/>
+      </material>
+    </visual>
+    <collision>
+      <geometry>
+        <cylinder radius="${wheel_radius}" length="${wheel_width}"/>
+      </geometry>
+    </collision>
+    <inertial>
+      <mass value="${wheel_mass}"/>
+      <inertia
+        ixx="0.01"
+        ixy="0.0"
+        ixz="0.0"
+        iyy="0.01"
+        iyz="0.0"
+        izz="0.01"/>
+    </inertial>
+  </link>
+  <joint name="left_wheel_joint" type="continuous">
+    <parent link="base_link"/>
+    <child link="left_wheel_link"/>
+    <origin xyz="0 0.325 -0.10" rpy="1.5708 0 0"/>
+    <axis xyz="0 0 1"/>
+  </joint>
+  <!-- ====================================================== -->
+  <!-- RIGHT DRIVE WHEEL                                      -->
+  <!-- ====================================================== -->
+  <link name="right_wheel_link">
+    <visual>
+      <geometry>
+        <cylinder radius="${wheel_radius}" length="${wheel_width}"/>
+      </geometry>
+      <material name="black">
+        <color rgba="0.05 0.05 0.05 1"/>
+      </material>
+    </visual>
+    <collision>
+      <geometry>
+        <cylinder radius="${wheel_radius}" length="${wheel_width}"/>
+      </geometry>
+    </collision>
+    <inertial>
+      <mass value="${wheel_mass}"/>
+      <inertia
+        ixx="0.01"
+        ixy="0.0"
+        ixz="0.0"
+        iyy="0.01"
+        iyz="0.0"
+        izz="0.01"/>
+    </inertial>
+  </link>
+  <joint name="right_wheel_joint" type="continuous">
+    <parent link="base_link"/>
+    <child link="right_wheel_link"/>
+    <origin xyz="0 -0.325 -0.10" rpy="1.5708 0 0"/>
+    <axis xyz="0 0 1"/>
+  </joint>
+  <!-- ====================================================== -->
+  <!-- FRONT CASTER                                           -->
+  <!-- ====================================================== -->
+  <link name="front_caster_link">
+    <visual>
+      <geometry>
+        <sphere radius="${caster_radius}"/>
+      </geometry>
+      <material name="caster_gray">
+        <color rgba="0.4 0.4 0.4 1"/>
+      </material>
+    </visual>
+    <collision>
+      <geometry>
+        <sphere radius="${caster_radius}"/>
+      </geometry>
+    </collision>
+    <inertial>
+      <mass value="${caster_mass}"/>
+      <inertia
+        ixx="0.001"
+        ixy="0.0"
+        ixz="0.0"
+        iyy="0.001"
+        iyz="0.0"
+        izz="0.001"/>
+    </inertial>
+  </link>
+  <joint name="front_caster_joint" type="fixed">
+    <parent link="base_link"/>
+    <child link="front_caster_link"/>
+    <origin xyz="0.30 0 -0.15" rpy="0 0 0"/>
+  </joint>
+  <!-- ====================================================== -->
+  <!-- REAR CASTER                                            -->
+  <!-- ====================================================== -->
+  <link name="rear_caster_link">
+    <visual>
+      <geometry>
+        <sphere radius="${caster_radius}"/>
+      </geometry>
+      <material name="caster_gray">
+        <color rgba="0.4 0.4 0.4 1"/>
+      </material>
+    </visual>
+    <collision>
+      <geometry>
+        <sphere radius="${caster_radius}"/>
+      </geometry>
+    </collision>
+    <inertial>
+      <mass value="${caster_mass}"/>
+      <inertia
+        ixx="0.001"
+        ixy="0.0"
+        ixz="0.0"
+        iyy="0.001"
+        iyz="0.0"
+        izz="0.001"/>
+    </inertial>
+  </link>
+  <joint name="rear_caster_joint" type="fixed">
+    <parent link="base_link"/>
+    <child link="rear_caster_link"/>
+    <origin xyz="-0.30 0 -0.15" rpy="0 0 0"/>
+  </joint>
+  <!-- ====================================================== -->
+  <!-- LIDAR                                                  -->
+  <!-- ====================================================== -->
+  <link name="lidar_link">
+    <visual>
+      <geometry>
+        <cylinder radius="${lidar_radius}" length="${lidar_height}"/>
+      </geometry>
+      <material name="lidar_black">
+        <color rgba="0.05 0.05 0.05 1"/>
+      </material>
+    </visual>
+    <collision>
+      <geometry>
+        <cylinder radius="${lidar_radius}" length="${lidar_height}"/>
+      </geometry>
+    </collision>
+    <inertial>
+      <mass value="${lidar_mass}"/>
+      <inertia
+        ixx="0.0001"
+        ixy="0.0"
+        ixz="0.0"
+        iyy="0.0001"
+        iyz="0.0"
+        izz="0.0001"/>
+    </inertial>
+  </link>
+  <joint name="lidar_joint" type="fixed">
+    <parent link="base_link"/>
+    <child link="lidar_link"/>
+    <origin xyz="0.20 0 0.14" rpy="0 0 0"/>
+  </joint>
+  <!-- ====================================================== -->
+  <!-- IMU                                                    -->
+  <!-- ====================================================== -->
+  <link name="imu_link">
+    <visual>
+      <geometry>
+        <box size="0.04 0.04 0.02"/>
+      </geometry>
+      <material name="imu_green">
+        <color rgba="0.1 0.8 0.2 1"/>
+      </material>
+    </visual>
+    <collision>
+      <geometry>
+        <box size="0.04 0.04 0.02"/>
+      </geometry>
+    </collision>
+    <inertial>
+      <mass value="${imu_mass}"/>
+      <inertia
+        ixx="0.00001"
+        ixy="0.0"
+        ixz="0.0"
+        iyy="0.00001"
+        iyz="0.0"
+        izz="0.00001"/>
+    </inertial>
+  </link>
+  <joint name="imu_joint" type="fixed">
+    <parent link="base_link"/>
+    <child link="imu_link"/>
+    <origin xyz="0 0 0.12" rpy="0 0 0"/>
+  </joint>
+  <!-- ====================================================== -->
+  <!-- GAZEBO DIFFERENTIAL DRIVE                              -->
+  <!-- ====================================================== -->
+  <gazebo>
+    <plugin filename="gz-sim-diff-drive-system"
+            name="gz::sim::systems::DiffDrive">
+      <left_joint>left_wheel_joint</left_joint>
+      <right_joint>right_wheel_joint</right_joint>
+      <wheel_separation>${wheel_separation}</wheel_separation>
+      <wheel_radius>${wheel_radius}</wheel_radius>
+      <topic>/cmd_vel</topic>
+      <odom_topic>/odom_raw</odom_topic>
+      <frame_id>odom</frame_id>
+      <child_frame_id>base_footprint</child_frame_id>
+      <odom_publish_frequency>50</odom_publish_frequency>
+    </plugin>
+  </gazebo>
+  <!-- ====================================================== -->
+  <!-- GAZEBO JOINT STATE PUBLISHER                           -->
+  <!-- ====================================================== -->
+  <gazebo>
+    <plugin filename="gz-sim-joint-state-publisher-system"
+            name="gz::sim::systems::JointStatePublisher">
+      <joint_name>left_wheel_joint</joint_name>
+      <joint_name>right_wheel_joint</joint_name>
+      <topic>/joint_states</topic>
+    </plugin>
+  </gazebo>
+  <!-- ====================================================== -->
+  <!-- GAZEBO LIDAR SENSOR                                    -->
+  <!-- ====================================================== -->
+  <gazebo reference="lidar_link">
     <sensor name="lidar_sensor" type="gpu_lidar">
-        <pose>0 0 0 0 0 0</pose>
-        <topic>/scan</topic>
-        <update_rate>10</update_rate>
-        <always_on>true</always_on>
-        <visualize>true</visualize>
-        <lidar>
-            <scan>
-                <horizontal>
-                    <samples>720</samples>
-                    <resolution>1</resolution>
-                    <min_angle>-3.14159265</min_angle>
-                    <max_angle>3.14159265</max_angle>
-                </horizontal>
-            </scan>
-            <range>
-                <min>0.10</min>
-                <max>10.0</max>
-                <resolution>0.01</resolution>
-            </range>
-        </lidar>
+      <pose>0 0 0 0 0 0</pose>
+      <topic>/scan</topic>
+      <update_rate>10</update_rate>
+      <always_on>true</always_on>
+      <visualize>true</visualize>
+      <lidar>
+        <scan>
+          <horizontal>
+            <samples>720</samples>
+            <resolution>1</resolution>
+            <min_angle>-3.14159265</min_angle>
+            <max_angle>3.14159265</max_angle>
+          </horizontal>
+        </scan>
+        <range>
+          <min>0.10</min>
+          <max>10.0</max>
+          <resolution>0.01</resolution>
+        </range>
+      </lidar>
     </sensor>
-</gazebo>
-<!-- ====================================================== -->
-<!-- LIDAR                                                  -->
-<!-- ====================================================== -->
-<xacro:property name="lidar_radius" value="0.05"/>
-<xacro:property name="lidar_height" value="0.04"/>
-<link name="lidar_link">
-    <visual>
-        <geometry>
-            <cylinder
-                radius="${lidar_radius}"
-                length="${lidar_height}"/>
-        </geometry>
-        <material name="lidar_black">
-            <color rgba="0.05 0.05 0.05 1"/>
-        </material>
-    </visual>
-    <collision>
-        <geometry>
-            <cylinder
-                radius="${lidar_radius}"
-                length="${lidar_height}"/>
-        </geometry>
-    </collision>
-    <inertial>
-        <mass value="0.2"/>
-        <inertia
-            ixx="0.0001"
-            ixy="0"
-            ixz="0"
-            iyy="0.0001"
-            iyz="0"
-            izz="0.0001"/>
-    </inertial>
-</link>
-<joint name="lidar_joint" type="fixed">
-    <parent link="base_link"/>
-    <child link="lidar_link"/>
-    <!-- Mounted on top of chassis -->
-    <origin
-        xyz="0.20 0 0.14"
-        rpy="0 0 0"/>
-</joint>
-<!-- ====================================================== -->
-<!-- IMU                                                    -->
-<!-- ====================================================== -->
-<link name="imu_link">
-    <visual>
-        <geometry>
-            <box size="0.04 0.04 0.02"/>
-        </geometry>
-        <material name="imu_green">
-            <color rgba="0.1 0.8 0.2 1"/>
-        </material>
-    </visual>
-    <collision>
-        <geometry>
-            <box size="0.04 0.04 0.02"/>
-        </geometry>
-    </collision>
-    <inertial>
-        <mass value="0.05"/>
-        <inertia
-            ixx="0.00001"
-            ixy="0"
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
Commit message: []

File: src/wms_description/urdf/wms_robot.urdf.xacro (robot description, xacro)
@@ -170,6 +170,11 @@
     <parent link="base_link"/>
     <child link="lidar_link"/>
+    <origin xyz="0.20 0 0.75" rpy="0 0 0"/>
+  </joint>
+  <!-- <joint name="lidar_joint" type="fixed">
+    <parent link="base_link"/>
+    <child link="lidar_link"/>
     <origin xyz="0.20 0 0.14" rpy="0 0 0"/>
-  </joint>
+  </joint> -->
   <!-- ====================================================== -->
   <!-- IMU                                                    -->
